File: pcb/pcb.kicad_pcb (KiCad board)
At the start: 2 copper layers, 66 x 61 mm, 16 parts, among them J1 GND, J2 HC-SR04, J3 PWM, J4 GPS UART, J5 Power Module v1.0, J6 UART, SW1 Reset, SW2 Action, U1 Pico, U2 NRF24L01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

Commit message: More sweeping changes, soon IO will be done?
Connections:
- J5 pad 1: Net-(J5-Pad1) -> GND
- J5 pad 2: Net-(J5-Pad1) -> GND
- J5 pad 5: GND -> Net-(J5-Pad5)
- J5 pad 6: GND -> Net-(J5-Pad5)
- U1 pad 31: Net-(J5-Pad4) -> Net-(J5-Pad3)
- U1 pad 32: Net-(J5-Pad3) -> Net-(J5-Pad4)
- U1 pad 39: Net-(J5-Pad1) -> Net-(J5-Pad5)
Routing:
- net Net-(J5-Pad1): track 16.0 -> 0.00 mm
- net Net-(J5-Pad5): track 0.00 -> 10.8 mm
- net Net-(J5-Pad4): track 28.8 -> 21.1 mm
- net GND: track 253.8 -> 261.1 mm
- net Net-(J5-Pad3): track 21.6 -> 25.1 mm

Commit message: Refactored organization
Connections:
- J5 pad 1: GND -> Net-(J5-Pad1)
- J5 pad 2: GND -> Net-(J5-Pad1)
- J5 pad 5: Net-(J5-Pad5) -> GND
- J5 pad 6: Net-(J5-Pad5) -> GND
- U1 pad 31: Net-(J5-Pad3) -> Net-(J5-Pad4)
- U1 pad 32: Net-(J5-Pad4) -> Net-(J5-Pad3)
- U1 pad 39: Net-(J5-Pad5) -> Net-(J5-Pad1)
Routing:
- net Net-(J5-Pad1): track 0.00 -> 16.0 mm
- net Net-(J5-Pad5): track 10.8 -> 0.00 mm
- net GND: track 261.1 -> 252.5 mm
- net Net-(J5-Pad4): track 21.1 -> 27.6 mm
- net Net-(J5-Pad3): track 25.1 -> 22.1 mm
